File: Surge.kicad_pcb (KiCad board)
At the start: 2 copper layers, 62.6 x 33.4 mm, 16 parts, among them SW1 ResetSW_Neon

Commit message: Refined Layout
Parts:
- SW1: value ResetSW_Neon -> C1005B 10A TCB
- turned SW1 to 0 degrees
Connections:
- F1 pad 2: Net-(SW1A-C) -> Net-(SW1A-A)
- H1 pad 1: Net-(SW1A-C) -> Net-(SW1A-A)
- H2 pad 1: Net-(SW1A-A) -> Net-(SW1A-C)
Other:
- outline, holes or cut-outs redrawn
Changed lines of the file:
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@@
   )
   (footprint "Surge_Library:Switch" (layer "F.Cu")
-    (at 52.3 50.35 180)
+    (at 52.3 50.35)
     (property "Sheetfile" "Surge.kicad_sch")
     (property "Sheetname" "")
@@
     (property "ki_keywords" "switch dual-pole double-throw DPDT spdt ON-ON")
     (attr smd)
-    (fp_text reference "SW1" (at 0 -0.5 180 unlocked) (layer "F.SilkS") hide
-        (effects (font (size 1 1) (thickness 0.1)))
-    )
-    (fp_text value "ResetSW_Neon" (at 0 1 180 unlocked) (layer "F.Fab") hide
-        (effects (font (size 1 1) (thickness 0.15)))
-    )
-    (fp_text user "${REFERENCE}" (at 0 2.5 180 unlocked) (layer "F.Fab")
+    (fp_text reference "SW1" (at 0 -0.5 unlocked) (layer "F.SilkS") hide
+        (effects (font (size 1 1) (thickness 0.1)))
+    )
+    (fp_text value "C1005B 10A TCB" (at 0 1 unlocked) (layer "F.Fab") hide
+        (effects (font (size 1 1) (thickness 0.15)))
+    )
+    (fp_text user "${REFERENCE}" (at 0 2.5 unlocked) (layer "F.Fab")
         (effects (font (size 1 1) (thickness 0.15)))
     )
@@
     (fp_line (start 7.5 11) (end -7.5 11)
       (stroke (width 0.1) (type default)) (layer "B.CrtYd"))
-    (pad "1" thru_hole roundrect (at 0 -6.6 180) (size 10 4.5) (drill oval 8 1.732) (layers "*.Cu" "*.Mask") (remove_unused_layers) (zone_layer_connections "F.Cu") (roundrect_rratio 0.25)
+    (pad "1" thru_hole roundrect (at 0 -6.6) (size 10 4.5) (drill oval 8 1.732) (layers "*.Cu" "*.Mask") (remove_unused_layers) (zone_layer_connections "F.Cu") (roundrect_rratio 0.25)
       (net 6 "Net-(SW1A-A)") (pinfunction "A") (pintype "passive") (thermal_bridge_angle 45))
-    (pad "2" thru_hole roundrect (at 0 0 180) (size 10 4.5) (drill oval 8 1.732) (layers "*.Cu" "*.Mask") (remove_unused_layers) (zone_layer_connections "F.Cu") (roundrect_rratio 0.25)
+    (pad "2" thru_hole roundrect (at 0 0) (size 10 4.5) (drill oval 8 1.732) (layers "*.Cu" "*.Mask") (remove_unused_layers) (zone_layer_connections "F.Cu") (roundrect_rratio 0.25)
       (net 4 "Net-(SW1A-B)") (pinfunction "B") (pintype "passive") (thermal_bridge_angle 45))
-    (pad "3" thru_hole roundrect (at 0 6.6 180) (size 10 4.5) (drill oval 8 1.732) (layers "*.Cu" "*.Mask") (remove_unused_layers) (zone_layer_connections "F.Cu") (roundrect_rratio 0.25)
+    (pad "3" thru_hole roundrect (at 0 6.6) (size 10 4.5) (drill oval 8 1.732) (layers "*.Cu" "*.Mask") (remove_unused_layers) (zone_layer_connections "F.Cu") (roundrect_rratio 0.25)
       (net 2 "Net-(SW1A-C)") (pinfunction "C") (pintype "passive") (thermal_bridge_angle 45))
   )
@@
     )
     (pad "1" thru_hole roundrect (at 0 -4.7) (size 5 5) (drill 2.8) (layers "*.Cu" "*.Mask") (remove_unused_layers) (zone_layer_connections "F.Cu") (roundrect_rratio 0.25)
-      (net 6 "Net-(SW1A-A)") (pinfunction "1") (pintype "input"))
+      (net 2 "Net-(SW1A-C)") (pinfunction "1") (pintype "input"))
   )
   (footprint "Surge_Library:L_Hole" (layer "F.Cu")
@@
     )
     (pad "1" thru_hole roundrect (at 0 -4.7) (size 5 5) (drill 2.8) (layers "*.Cu" "*.Mask") (remove_unused_layers) (zone_layer_connections "F.Cu") (roundrect_rratio 0.25)
-      (net 2 "Net-(SW1A-C)") (pinfunction "1") (pintype "input"))
+      (net 6 "Net-(SW1A-A)") (pinfunction "1") (pintype "input"))
   )
   (footprint "Varistor:RV_Disc_D21.5mm_W4.7mm_P10mm" (layer "B.Cu")
@@
       (net 1 "Net-(F1-Pad1)") (pintype "passive"))
     (pad "2" thru_hole circle (at 7.5 0 180) (size 2 2) (drill 1) (layers "*.Cu" "*.Mask") (remove_unused_layers) (zone_layer_connections "F.Cu")
-      (net 2 "Net-(SW1A-C)") (pintype "passive"))
+      (net 6 "Net-(SW1A-A)") (pintype "passive"))
     (model "${KICAD6_3DMODEL_DIR}/Capacitor_THT.3dshapes/C_Rect_L10.3mm_W5.0mm_P7.50mm_MKS4.wrl"
       (offset (xyz 0 0 0))
@@
   (gr_line (start 71.025735 61.6) (end 71.352467 61.6)
     (stroke (width 0.1) (type default)) (layer "Edge.Cuts"))
-  (gr_circle (center 39.64 50.2) (end 40.51 50.2)
-    (stroke (width 0.1) (type default)) (fill none) (layer "Edge.Cuts"))
   (gr_line (start 96.77 52.79) (end 78.53 52.79)
     (stroke (width 0.1) (type default)) (layer "Edge.Cuts"))
@@
     (polygon
       (pts
-        (xy 37.175 62.55)
-        (xy 36.3 63.425)
-        (xy 36.3 68)
-        (xy 36.9 68.6)
+        (xy 37.675 62.55)
+        (xy 36.53 63.695)
+        (xy 36.53 67.54)
+        (xy 37.59 68.6)
         (xy 62.625 68.6)
         (xy 64.25 66.975)
@@
     (polygon
       (pts
-        (xy 78.175 36.4)
+        (xy 77.815 36.76)
         (xy 76.15 38.425)
         (xy 76.15 47.95)
-        (xy 79.125 50.925)
-        (xy 96.36 50.925)
-        (xy 97.98 49.305)
-        (xy 97.98 37.97)
-        (xy 96.41 36.4)
+        (xy 78.895 50.695)
+        (xy 96.39 50.695)
+        (xy 97.62 49.465)
+        (xy 97.62 38.06)
+        (xy 96.32 36.76)
       )
     )
@@
     (polygon
       (pts
-        (xy 76.575 53.325)
+        (xy 76.405 53.495)
         (xy 76.075 53.825)
         (xy 76.075 66.8)
-        (xy 77.925 68.65)
-        (xy 95.985 68.65)
-        (xy 98.005 66.63)
-        (xy 98.005 55.13)
-        (xy 96.2 53.325)
+        (xy 77.705 68.43)
+        (xy 96.205 68.43)
+        (xy 97.605 67.03)
+        (xy 97.605 54.73)
+        (xy 96.37 53.495)
       )
     )
   )
-  (zone (net 6) (net_name "Net-(SW1A-A)") (layer "F.Cu") (hatch edge 0.5)
+  (zone (net 2) (net_name "Net-(SW1A-C)") (layer "F.Cu") (hatch edge 0.5)
     (priority 2)
     (connect_pads yes (clearance 0.5))
@@
     (polygon
       (pts
-        (xy 37.2 54.4)
-        (xy 36.35 55.25)
-        (xy 36.35 59.225)
-        (xy 37.25 60.125)
+        (xy 37.51 54.4)
+        (xy 36.54 55.37)
+        (xy 36.54 59.115)
+        (xy 37.55 60.125)
         (xy 56.925 60.125)
         (xy 57.525 59.525)
@@
     )
   )
-  (zone (net 2) (net_name "Net-(SW1A-C)") (layer "F.Cu") (hatch edge 0.5)
+  (zone (net 6) (net_name "Net-(SW1A-A)") (layer "F.Cu") (hatch edge 0.5)
     (connect_pads yes (clearance 0.5))
     (min_thickness 0.25) (filled_areas_thickness no)
@@
     (polygon
       (pts
-        (xy 37.429724 40.25)
-        (xy 36.393986 41.285738)
-        (xy 36.365781 45.520781)
-        (xy 37.12 46.275)
+        (xy 37.889724 40.25)
+        (xy 36.749763 41.389961)
+        (xy 36.724856 45.129856)
+        (xy 37.87 46.275)
         (xy 64.230147 46.275)
         (xy 65.383059 47.469874)

Commit message: update layout
Parts:
- removed NE6: E_E, Surge_Library:NEmount
- added NE4: , Surge_Library:NEmount, F.Cu at (59.9, 31.2)
- NE5: value E_MOV -> (none)
- SW1: moved to B.Cu
- moved H3 36.1 mm to (36.4, 34.3)
- moved H6 36.0 mm to (59.9, 29.5)
- moved NE5 22.0 mm to (60.0, 62.3)
- moved H5 7.88 mm to (84.8, 62.0)
- moved H4 7.00 mm to (85.0, 45.1)
- moved F1 7.00 mm to (74.5, 38.4)
- moved F2 7.00 mm to (74.5, 49.2)
- moved RV1 7.00 mm to (65.9, 34.0)
- moved RV2 7.00 mm to (65.9, 44.8)
- moved RV3 7.00 mm to (75.9, 53.6)
- moved NE3 6.70 mm to (81.3, 52.5)
- moved NE2 6.70 mm to (81.3, 40.9)
- moved H1 5.38 mm to (37.1, 43.2)
- moved SW1 3.09 mm to (49.9, 48.4), turned to 180 degrees
- moved H2 2.92 mm to (36.6, 63.1)
Connections:
- RV1 pad 2: Net-(NE5-Pad1) -> Earth
- RV3 pad 2: Earth -> Net-(NE5-Pad1)
Routing:
- net Earth: track 9.66 -> 0.00 mm
- net Net-(NE5-Pad1): track 8.76 -> 7.64 mm
Other:
- board size 62.6 x 33.4 mm -> 61.6 x 36.2 mm
- board text added: "TCB"
- board text removed: "SPST_Neon SW"
