File: Surge.kicad_pcb (KiCad board)
At the start: 2 copper layers, 61.6 x 36.2 mm, 16 parts, among them SW1 C1005B 10A TCB

Commit message: Update Schematics
Parts:
- RV1, RV2, RV3: value 471KD20J -> 471K
- moved H3 0.62 mm to (37.0, 34.3)
- moved H2 0.42 mm to (37.0, 63.1)
- moved H1 0.07 mm to (37.0, 43.2)
- renumbered NE5 to J1, NE4 to J2
Other:
- outline, holes or cut-outs redrawn

Commit message: Update Readme
Parts:
- renumbered NE2 to NE1, NE3 to NE2
Changed lines of the file:
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@@
     (property "ki_keywords" "test point tp")
     (attr smd exclude_from_bom)
-    (fp_text reference "NE3" (at 0 -0.5 unlocked) (layer "User.1")
+    (fp_text reference "NE2" (at 0 -0.5 unlocked) (layer "User.1")
         (effects (font (size 1 1) (thickness 0.1)))
     )
@@
     (property "ki_keywords" "test point tp")
     (attr smd exclude_from_bom)
-    (fp_text reference "NE2" (at 0 -0.5 unlocked) (layer "User.1")
+    (fp_text reference "NE1" (at 0 -0.5 unlocked) (layer "User.1")
         (effects (font (size 1 1) (thickness 0.1)))
     )

Commit message: Update BOM and ReadMe
Parts:
- SW1: value C1005B 10A TCB -> C1005B 15A TCB
