File: Surge.kicad_sch (KiCad schematic)
At the start: 14 parts, among them SW1 SW_DPDT_x2

Commit message: update values
Parts:
- F1, F2: value Fuse -> 115C 20A 250V
- R1: value R -> 200K Ω
- RV1, RV2, RV3: value Varistor -> 471KD20J
Changed lines of the file:
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@@
   (symbol (lib_id "Device:Fuse") (at 68.58 30.48 270) (unit 1)
     (in_bom yes) (on_board yes) (dnp no) (fields_autoplaced)
-    (property "Reference" "F1" (at 68.58 25.5737 90)
-      (effects (font (size 1.27 1.27)))
-    )
-    (property "Value" "Fuse" (at 68.58 27.9979 90)
-      (effects (font (size 1.27 1.27)))
+    (property "Reference" "F1" (at 68.58 25.4 90)
+      (effects (font (size 1.27 1.27)))
+    )
+    (property "Value" "115C 20A 250V" (at 68.58 26.67 90)
+      (effects (font (size 1 1)))
     )
     (property "Footprint" "" (at 68.58 28.702 90)
@@
   )
   (symbol (lib_id "Device:R") (at 83.82 43.18 270) (unit 1)
-    (in_bom yes) (on_board yes) (dnp no) (fields_autoplaced)
-    (property "Reference" "R1" (at 83.82 38.0197 90)
-      (effects (font (size 1.27 1.27)))
-    )
-    (property "Value" "R" (at 83.82 40.4439 90)
-      (effects (font (size 1.27 1.27)))
+    (in_bom yes) (on_board yes) (dnp no)
+    (property "Reference" "R1" (at 83.82 38.1 90)
+      (effects (font (size 1.27 1.27)))
+    )
+    (property "Value" "200K Ω" (at 83.82 40.64 90)
+      (effects (font (size 1 1)))
     )
     (property "Footprint" "" (at 83.82 41.402 90)
@@
   (symbol (lib_id "Device:Varistor") (at 100.33 57.15 0) (unit 1)
     (in_bom yes) (on_board yes) (dnp no) (fields_autoplaced)
-    (property "Reference" "RV3" (at 102.87 56.1312 0)
+    (property "Reference" "RV3" (at 102.87 56.0733 0)
       (effects (font (size 1.27 1.27)) (justify left))
     )
-    (property "Value" "Varistor" (at 102.87 58.5554 0)
-      (effects (font (size 1.27 1.27)) (justify left))
+    (property "Value" "471KD20J" (at 102.87 58.6132 0)
+      (effects (font (size 1 1)) (justify left))
     )
     (property "Footprint" "" (at 98.552 57.15 90)
@@
   (symbol (lib_id "Device:Varistor") (at 100.33 41.91 180) (unit 1)
     (in_bom yes) (on_board yes) (dnp no) (fields_autoplaced)
-    (property "Reference" "RV1" (at 103.5194 40.5046 0)
+    (property "Reference" "RV1" (at 104.14 40.4467 0)
       (effects (font (size 1.27 1.27)) (justify right))
     )
-    (property "Value" "Varistor" (at 103.5194 42.9288 0)
-      (effects (font (size 1.27 1.27)) (justify right))
+    (property "Value" "471KD20J" (at 104.14 42.9866 0)
+      (effects (font (size 1 1)) (justify right))
     )
     (property "Footprint" "" (at 102.108 41.91 90)
@@
   (symbol (lib_id "Device:Varistor") (at 100.33 25.4 0) (unit 1)
     (in_bom yes) (on_board yes) (dnp no) (fields_autoplaced)
-    (property "Reference" "RV2" (at 102.87 24.3812 0)
+    (property "Reference" "RV2" (at 102.87 24.3233 0)
       (effects (font (size 1.27 1.27)) (justify left))
     )
-    (property "Value" "Varistor" (at 102.87 26.8054 0)
-      (effects (font (size 1.27 1.27)) (justify left))
+    (property "Value" "471KD20J" (at 102.87 26.8632 0)
+      (effects (font (size 1 1)) (justify left))
     )
     (property "Footprint" "" (at 98.552 25.4 90)
@@
       (effects (font (size 1.27 1.27)))
     )
-    (property "Value" "Fuse" (at 68.58 49.5879 90)
-      (effects (font (size 1.27 1.27)))
+    (property "Value" "115C 20A 250V" (at 68.58 49.5879 90)
+      (effects (font (size 1 1)))
     )
     (property "Footprint" "" (at 68.58 50.292 90)

Commit message: update footprints
Parts:
- F1, F2: value 115C 20A 250V -> TCO 115C 20A 250V; footprint (none) -> Capacitor_THT:C_Rect_L10.3mm_W5.0mm_P7.50mm_MKS4
- H1, H5: footprint (none) -> Surge_Library:I_Hole
- H2: value L_in -> N_in; footprint (none) -> Surge_Library:I_Hole
- H3: value N_out -> L_out; footprint (none) -> Surge_Library:L_Hole
- H4: value L_out -> N_out; footprint (none) -> Surge_Library:L_Hole
- H6: footprint (none) -> Surge_Library:L_Hole
- NE1: footprint (none) -> Surge_Library:NE2
- R1: footprint (none) -> Resistor_THT:R_Axial_DIN0414_L11.9mm_D4.5mm_P15.24mm_Horizontal
- RV1, RV2, RV3: footprint (none) -> Varistor:RV_Disc_D21.5mm_W4.7mm_P10mm
- SW1: value SW_DPDT_x2 -> ResetSW_Neon; footprint (none) -> Surge_Library:Switch
Changed lines of the file:
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@@
   (symbol (lib_id "Mechanical:MountingHole_Pad") (at 33.02 52.07 90) (unit 1)
     (in_bom yes) (on_board yes) (dnp no) (fields_autoplaced)
-    (property "Reference" "H2" (at 31.75 46.1477 90)
-      (effects (font (size 1.27 1.27)))
-    )
-    (property "Value" "L_in" (at 31.75 48.5719 90)
-      (effects (font (size 1.27 1.27)))
-    )
-    (property "Footprint" "" (at 33.02 52.07 0)
+    (property "Reference" "H2" (at 31.75 45.72 90)
+      (effects (font (size 1.27 1.27)))
+    )
+    (property "Value" "N_in" (at 31.75 48.26 90)
+      (effects (font (size 1.27 1.27)))
+    )
+    (property "Footprint" "Surge_Library:I_Hole" (at 33.02 52.07 0)
       (effects (font (size 1.27 1.27)) hide)
     )
@@
   (symbol (lib_id "Mechanical:MountingHole_Pad") (at 111.76 52.07 270) (unit 1)
     (in_bom yes) (on_board yes) (dnp no) (fields_autoplaced)
-    (property "Reference" "H4" (at 115.57 50.8579 90)
-      (effects (font (size 1.27 1.27)) (justify left))
-    )
-    (property "Value" "L_out" (at 115.57 53.2821 90)
-      (effects (font (size 1.27 1.27)) (justify left))
-    )
-    (property "Footprint" "" (at 111.76 52.07 0)
+    (property "Reference" "H4" (at 115.57 50.8 90)
+      (effects (font (size 1.27 1.27)) (justify left))
+    )
+    (property "Value" "N_out" (at 115.57 53.34 90)
+      (effects (font (size 1.27 1.27)) (justify left))
+    )
+    (property "Footprint" "Surge_Library:L_Hole" (at 111.76 52.07 0)
       (effects (font (size 1.27 1.27)) hide)
     )
@@
   )
   (symbol (lib_id "Device:Fuse") (at 68.58 30.48 270) (unit 1)
-    (in_bom yes) (on_board yes) (dnp no) (fields_autoplaced)
+    (in_bom yes) (on_board yes) (dnp no)
     (property "Reference" "F1" (at 68.58 25.4 90)
       (effects (font (size 1.27 1.27)))
     )
-    (property "Value" "115C 20A 250V" (at 68.58 26.67 90)
+    (property "Value" "TCO 115C 20A 250V" (at 68.58 27.94 90)
       (effects (font (size 1 1)))
     )
-    (property "Footprint" "" (at 68.58 28.702 90)
+    (property "Footprint" "Capacitor_THT:C_Rect_L10.3mm_W5.0mm_P7.50mm_MKS4" (at 68.58 28.702 90)
       (effects (font (size 1.27 1.27)) hide)
     )
@@
       (effects (font (size 1 1)))
     )
-    (property "Footprint" "" (at 83.82 41.402 90)
+    (property "Footprint" "Resistor_THT:R_Axial_DIN0414_L11.9mm_D4.5mm_P15.24mm_Horizontal" (at 83.82 41.402 90)
       (effects (font (size 1.27 1.27)) hide)
     )
@@
       (effects (font (size 1 1)) (justify left))
     )
-    (property "Footprint" "" (at 98.552 57.15 90)
+    (property "Footprint" "Varistor:RV_Disc_D21.5mm_W4.7mm_P10mm" (at 98.552 57.15 90)
       (effects (font (size 1.27 1.27)) hide)
     )
@@
       (effects (font (size 1.27 1.27)))
     )
-    (property "Footprint" "" (at 67.31 43.18 90)
+    (property "Footprint" "Surge_Library:NE2" (at 67.31 43.18 90)
       (effects (font (size 1.27 1.27)) hide)
     )
@@
       (effects (font (size 1.27 1.27)))
     )
-    (property "Footprint" "" (at 119.38 43.18 0)
+    (property "Footprint" "Surge_Library:L_Hole" (at 119.38 43.18 0)
       (effects (font (size 1.27 1.27)) hide)
     )
@@
       (effects (font (size 1.27 1.27)))
     )
-    (property "Footprint" "" (at 33.02 30.48 0)
+    (property "Footprint" "Surge_Library:I_Hole" (at 33.02 30.48 0)
       (effects (font (size 1.27 1.27)) hide)
     )
@@
       (effects (font (size 1 1)) (justify right))
     )
-    (property "Footprint" "" (at 102.108 41.91 90)
+    (property "Footprint" "Varistor:RV_Disc_D21.5mm_W4.7mm_P10mm" (at 102.108 41.91 90)
       (effects (font (size 1.27 1.27)) hide)
     )
@@
   (symbol (lib_id "Switch:SW_DPDT_x2") (at 50.8 43.18 180) (unit 1)
     (in_bom yes) (on_board yes) (dnp no) (fields_autoplaced)
-    (property "Reference" "SW1" (at 50.8 36.1147 0)
-      (effects (font (size 1.27 1.27)))
-    )
-    (property "Value" "SW_DPDT_x2" (at 50.8 38.5389 0)
-      (effects (font (size 1.27 1.27)))
-    )
-    (property "Footprint" "" (at 50.8 43.18 0)
+    (property "Reference" "SW1" (at 50.8 35.56 0)
+      (effects (font (size 1.27 1.27)))
+    )
+    (property "Value" "ResetSW_Neon" (at 50.8 38.1 0)
+      (effects (font (size 1.27 1.27)))
+    )
+    (property "Footprint" "Surge_Library:Switch" (at 50.8 43.18 0)
       (effects (font (size 1.27 1.27)) hide)
     )
@@
       (effects (font (size 1 1)) (justify left))
     )
-    (property "Footprint" "" (at 98.552 25.4 90)
+    (property "Footprint" "Varistor:RV_Disc_D21.5mm_W4.7mm_P10mm" (at 98.552 25.4 90)
       (effects (font (size 1.27 1.27)) hide)
     )
@@
       (effects (font (size 1.27 1.27)))
     )
-    (property "Footprint" "" (at 33.02 62.23 0)
+    (property "Footprint" "Surge_Library:I_Hole" (at 33.02 62.23 0)
       (effects (font (size 1.27 1.27)) hide)
     )
@@
   (symbol (lib_id "Mechanical:MountingHole_Pad") (at 111.76 30.48 270) (unit 1)
     (in_bom yes) (on_board yes) (dnp no) (fields_autoplaced)
-    (property "Reference" "H3" (at 115.57 29.2679 90)
-      (effects (font (size 1.27 1.27)) (justify left))
-    )
-    (property "Value" "N_out" (at 115.57 31.6921 90)
-      (effects (font (size 1.27 1.27)) (justify left))
-    )
-    (property "Footprint" "" (at 111.76 30.48 0)
+    (property "Reference" "H3" (at 115.57 29.21 90)
+      (effects (font (size 1.27 1.27)) (justify left))
+    )
+    (property "Value" "L_out" (at 115.57 31.75 90)
+      (effects (font (size 1.27 1.27)) (justify left))
+    )
+    (property "Footprint" "Surge_Library:L_Hole" (at 111.76 30.48 0)
       (effects (font (size 1.27 1.27)) hide)
     )
@@
       (effects (font (size 1.27 1.27)))
     )
-    (property "Value" "115C 20A 250V" (at 68.58 49.5879 90)
+    (property "Value" "TCO 115C 20A 250V" (at 68.58 49.5879 90)
       (effects (font (size 1 1)))
     )
-    (property "Footprint" "" (at 68.58 50.292 90)
-      (effects (font (size 1.27 1.27)) hide)
-    )
+    (property "Footprint" "Capacitor_THT:C_Rect_L10.3mm_W5.0mm_P7.50mm_MKS4" (at 68.58 50.292 90)
+      (effects (font (size 1.27 1.27)) hide)
+    )

Commit message: Updated board layout
Parts:
- added NE2: NE_N, Surge_Library:NEmount, symbol Connector:TestPoint
- added NE3: NE_L, Surge_Library:NEmount, symbol Connector:TestPoint
- added NE5: E_MOV, Surge_Library:NEmount, symbol Connector:TestPoint
- added NE6: E_E, Surge_Library:NEmount, symbol Connector:TestPoint
- H1: value L_in -> N_in
- H2: value N_in -> L_in
- H4: renamed from H3; value L_out -> N_out
- H5: renamed from H4; value N_out -> L_out
- H6: footprint Surge_Library:L_Hole -> Surge_Library:I_Hole
- renumbered H5 to H3, RV2 to RV1, RV1 to RV2
Connections:
- net Earth: now also NE6.1; no longer RV1.1
- net at F2.1, H5.1, RV2.1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: now also NE3.1; no longer R1.1
- net at F1.1, H4.1, RV1.2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: now also NE2.1; no longer NE1.2
- new net: NE5.1, RV1.1
- no-connect marks 0 -> 2
Other:
- moved on the sheet: F2, H2, H3, H5, H6, NE1, R1, RV2, RV3, SW1A

Commit message: Updated board layout
Connections:
- net at F2.1, H5.1, NE3.1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: now also RV2.2; no longer RV2.1
- net at F1.1, H4.1, NE2.1: now also RV1.1, RV2.1; no longer RV1.2, RV2.2
- net at NE5.1: now also RV1.2; no longer RV1.1
Other:
- moved on the sheet: RV1, RV2
Changed lines of the file:
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@@
-    (stroke (width 0) (type default))
-  )
-  (wire (pts (xy 45.72 49.53) (xy 45.72 60.96))
     (stroke (width 0) (type default))
   )
@@
     (stroke (width 0) (type default))
   )
-  (wire (pts (xy 35.56 60.96) (xy 45.72 60.96))
+  (wire (pts (xy 45.72 60.96) (xy 45.72 49.53))
     (stroke (width 0) (type default))
   )
@@
   )
   (wire (pts (xy 55.88 46.99) (xy 55.88 60.96))
+    (stroke (width 0) (type default))
+  )
+  (wire (pts (xy 35.56 60.96) (xy 45.72 60.96))
     (stroke (width 0) (type default))
   )
@@
     )
   )
-  (symbol (lib_id "Device:Varistor") (at 100.33 45.72 180) (unit 1)
-    (in_bom yes) (on_board yes) (dnp no) (fields_autoplaced)
-    (property "Reference" "RV2" (at 104.14 44.2567 0)
-      (effects (font (size 1.27 1.27)) (justify right))
-    )
-    (property "Value" "471KD20J" (at 104.14 46.7966 0)
-      (effects (font (size 1 1)) (justify right))
-    )
-    (property "Footprint" "Varistor:RV_Disc_D21.5mm_W4.7mm_P10mm" (at 102.108 45.72 90)
+  (symbol (lib_id "Device:Varistor") (at 100.33 45.72 0) (unit 1)
+    (in_bom yes) (on_board yes) (dnp no) (fields_autoplaced)
+    (property "Reference" "RV2" (at 102.87 44.6433 0)
+      (effects (font (size 1.27 1.27)) (justify left))
+    )
+    (property "Value" "471KD20J" (at 102.87 47.1832 0)
+      (effects (font (size 1 1)) (justify left))
+    )
+    (property "Footprint" "Varistor:RV_Disc_D21.5mm_W4.7mm_P10mm" (at 98.552 45.72 90)
       (effects (font (size 1.27 1.27)) hide)
     )
@@
     )
   )
-  (symbol (lib_id "Device:Varistor") (at 100.33 25.4 0) (unit 1)
-    (in_bom yes) (on_board yes) (dnp no) (fields_autoplaced)
-    (property "Reference" "RV1" (at 102.87 24.3233 0)
-      (effects (font (size 1.27 1.27)) (justify left))
-    )
-    (property "Value" "471KD20J" (at 102.87 26.8632 0)
-      (effects (font (size 1 1)) (justify left))
-    )
-    (property "Footprint" "Varistor:RV_Disc_D21.5mm_W4.7mm_P10mm" (at 98.552 25.4 90)
-      (effects (font (size 1.27 1.27)) hide)
-    )
+  (symbol (lib_id "Device:Varistor") (at 100.33 25.4 180) (unit 1)
+    (in_bom yes) (on_board yes) (dnp no) (fields_autoplaced)
+    (property "Reference" "RV1" (at 104.14 23.9367 0)
+      (effects (font (size 1.27 1.27)) (justify right))
+    )
+    (property "Value" "471KD20J" (at 104.14 26.4766 0)
+      (effects (font (size 1 1)) (justify right))
+    )
+    (property "Footprint" "Varistor:RV_Disc_D21.5mm_W4.7mm_P10mm" (at 102.108 25.4 90)
+      (effects (font (size 1.27 1.27)) hide)
+    )

Commit message: Refined Layout
Parts:
- SW1: value ResetSW_Neon -> C1005B 10A TCB
Connections:
- net at H2.1: now also SW1.3 (C); no longer SW1.1 (A)
- net at F1.2, H1.1: now also SW1.1 (A); no longer SW1.3 (C)
Other:
- moved on the sheet: SW1A
Changed lines of the file:
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@@
     )
   )
-  (symbol (lib_id "Switch:SW_DPDT_x2") (at 50.8 46.99 180) (unit 1)
-    (in_bom yes) (on_board yes) (dnp no) (fields_autoplaced)
-    (property "Reference" "SW1" (at 50.8 39.37 0)
+  (symbol (lib_id "Switch:SW_DPDT_x2") (at 50.8 46.99 0) (mirror y) (unit 1)
+    (in_bom yes) (on_board yes) (dnp no)
+    (property "Reference" "SW1" (at 52.07 43.18 0)
       (effects (font (size 1.27 1.27)))
     )
-    (property "Value" "ResetSW_Neon" (at 50.8 41.91 0)
+    (property "Value" "C1005B 10A TCB" (at 52.07 40.64 0)
       (effects (font (size 1.27 1.27)))
     )

Commit message: update layout
Parts:
- removed NE6: E_E, Surge_Library:NEmount, symbol Connector:TestPoint
- added NE4: (no value), Surge_Library:NEmount, symbol Connector:TestPoint
- NE5: value E_MOV -> (none)
Connections:
- net Earth: now also RV1.2, NE4.1; no longer RV3.2
- net at NE5.1: now also RV3.2; no longer RV1.2
Other:
- moved on the sheet: H3
Changed lines of the file:
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@@
   (junction (at 100.33 60.96) (diameter 0) (color 0 0 0 0)
   )
-  (junction (at 100.33 71.12) (diameter 0) (color 0 0 0 0)
+  (junction (at 100.33 83.82) (diameter 0) (color 0 0 0 0)
   )
   (junction (at 86.36 30.48) (diameter 0) (color 0 0 0 0)
@@
     (stroke (width 0) (type default))
   )
-  (wire (pts (xy 100.33 20.32) (xy 106.68 20.32))
-    (stroke (width 0) (type default))
-  )
   (polyline (pts (xy 78.74 34.29) (xy 86.36 34.29))
     (stroke (width 0) (type dot))
@@
     (stroke (width 0) (type default))
   )
-  (wire (pts (xy 35.56 71.12) (xy 100.33 71.12))
+  (wire (pts (xy 35.56 83.82) (xy 100.33 83.82))
     (stroke (width 0) (type default))
   )
@@
   )
   (wire (pts (xy 41.91 30.48) (xy 64.77 30.48))
+    (stroke (width 0) (type default))
+  )
+  (wire (pts (xy 100.33 69.85) (xy 100.33 71.12))
     (stroke (width 0) (type default))
   )
@@
     (stroke (width 0) (type default))
   )
-  (wire (pts (xy 125.73 45.72) (xy 125.73 71.12))
+  (wire (pts (xy 100.33 81.28) (xy 100.33 83.82))
+    (stroke (width 0) (type default))
+  )
+  (wire (pts (xy 125.73 45.72) (xy 125.73 83.82))
     (stroke (width 0) (type default))
   )
@@
     (stroke (width 0) (type default))
   )
-  (wire (pts (xy 100.33 71.12) (xy 100.33 69.85))
-    (stroke (width 0) (type default))
-  )
-  (wire (pts (xy 125.73 71.12) (xy 100.33 71.12))
+  (wire (pts (xy 125.73 83.82) (xy 100.33 83.82))
     (stroke (width 0) (type default))
   )
@@
     (stroke (width 0) (type default))
   )
-  (polyline (pts (xy 107.95 20.32) (xy 120.65 20.32))
+  (wire (pts (xy 86.36 30.48) (xy 100.33 30.48))
+    (stroke (width 0) (type default))
+  )
+  (wire (pts (xy 72.39 60.96) (xy 86.36 60.96))
+    (stroke (width 0) (type default))
+  )
+  (wire (pts (xy 55.88 46.99) (xy 55.88 60.96))
+    (stroke (width 0) (type default))
+  )
+  (wire (pts (xy 35.56 60.96) (xy 45.72 60.96))
+    (stroke (width 0) (type default))
+  )
+  (polyline (pts (xy 100.33 78.74) (xy 100.33 73.66))
     (stroke (width 0) (type dot))
   )
-  (wire (pts (xy 86.36 30.48) (xy 100.33 30.48))
-    (stroke (width 0) (type default))
-  )
-  (wire (pts (xy 72.39 60.96) (xy 86.36 60.96))
-    (stroke (width 0) (type default))
-  )
-  (wire (pts (xy 55.88 46.99) (xy 55.88 60.96))
-    (stroke (width 0) (type default))
-  )
-  (wire (pts (xy 35.56 60.96) (xy 45.72 60.96))
-    (stroke (width 0) (type default))
-  )
-  (wire (pts (xy 121.92 20.32) (xy 125.73 20.32))
+  (wire (pts (xy 100.33 20.32) (xy 125.73 20.32))
     (stroke (width 0) (type default))
   )
@@
         (path "/87282895-5363-4673-9c65-8e036a00088a"
           (reference "NE1") (unit 1)
+        )
+      )
+    )
+  )
+  (symbol (lib_id "Connector:TestPoint") (at 100.33 71.12 180) (unit 1)
+    (in_bom no) (on_board yes) (dnp no)
+    (property "Reference" "NE5" (at 99.06 73.66 0)
+      (effects (font (size 1.27 1.27)) (justify left))
+    )
+    (property "Value" " " (at 99.06 74.93 0)
+      (effects (font (size 1.27 1.27)) (justify left))
+    )
+    (property "Footprint" "Surge_Library:NEmount" (at 95.25 71.12 0)
+      (effects (font (size 1.27 1.27)) hide)
+    )
+    (property "Datasheet" "~" (at 95.25 71.12 0)
+      (effects (font (size 1.27 1.27)) hide)
+    )
+    (pin "1")
+    (instances
+      (project "Surge"
+        (path "/87282895-5363-4673-9c65-8e036a00088a"
+          (reference "NE5") (unit 1)
+        )
+      )
+    )
+  )
+  (symbol (lib_id "Connector:TestPoint") (at 100.33 81.28 0) (unit 1)
+    (in_bom no) (on_board yes) (dnp no)
+    (property "Reference" "NE4" (at 99.06 78.74 0)
+      (effects (font (size 1.27 1.27)) (justify right))
+    )
+    (property "Value" " " (at 99.06 81.28 0)
+      (effects (font (size 1.27 1.27)) (justify right))
+    )
+    (property "Footprint" "Surge_Library:NEmount" (at 105.41 81.28 0)
+      (effects (font (size 1.27 1.27)) hide)
+    )
+    (property "Datasheet" "~" (at 105.41 81.28 0)
+      (effects (font (size 1.27 1.27)) hide)
+    )
+    (pin "1")
+    (instances
+      (project "Surge"
+        (path "/87282895-5363-4673-9c65-8e036a00088a"
+          (reference "NE4") (unit 1)
         )
       )
@@
     )
   )
-  (symbol (lib_id "power:Earth") (at 100.33 71.12 0) (unit 1)
-    (in_bom yes) (on_board yes) (dnp no) (fields_autoplaced)
-    (property "Reference" "#PWR01" (at 100.33 77.47 0)
-      (effects (font (size 1.27 1.27)) hide)
-    )
-    (property "Value" "Earth" (at 100.33 74.93 0)
-      (effects (font (size 1.27 1.27)) hide)
-    )
-    (property "Footprint" "" (at 100.33 71.12 0)
-      (effects (font (size 1.27 1.27)) hide)
-    )
-    (property "Datasheet" "~" (at 100.33 71.12 0)
+  (symbol (lib_id "power:Earth") (at 100.33 83.82 0) (unit 1)
+    (in_bom yes) (on_board yes) (dnp no) (fields_autoplaced)
+    (property "Reference" "#PWR01" (at 100.33 90.17 0)
+      (effects (font (size 1.27 1.27)) hide)
+    )
+    (property "Value" "Earth" (at 100.33 87.63 0)
+      (effects (font (size 1.27 1.27)) hide)
+    )
+    (property "Footprint" "" (at 100.33 83.82 0)
+      (effects (font (size 1.27 1.27)) hide)
+    )
+    (property "Datasheet" "~" (at 100.33 83.82 0)
       (effects (font (size 1.27 1.27)) hide)
     )
@@
     )
   )
-  (symbol (lib_id "Mechanical:MountingHole_Pad") (at 33.02 71.12 90) (unit 1)
-    (in_bom yes) (on_board yes) (dnp no) (fields_autoplaced)
-    (property "Reference" "H3" (at 31.75 65.1977 90)
-      (effects (font (size 1.27 1.27)))
-    )
-    (property "Value" "E_in" (at 31.75 67.6219 90)
-      (effects (font (size 1.27 1.27)))
-    )
-    (property "Footprint" "Surge_Library:I_Hole" (at 33.02 71.12 0)
-      (effects (font (size 1.27 1.27)) hide)
-    )
-    (property "Datasheet" "~" (at 33.02 71.12 0)
+  (symbol (lib_id "Mechanical:MountingHole_Pad") (at 33.02 83.82 90) (unit 1)
+    (in_bom yes) (on_board yes) (dnp no) (fields_autoplaced)
+    (property "Reference" "H3" (at 31.75 77.8977 90)
+      (effects (font (size 1.27 1.27)))
+    )
+    (property "Value" "E_in" (at 31.75 80.3219 90)
+      (effects (font (size 1.27 1.27)))
+    )
+    (property "Footprint" "Surge_Library:I_Hole" (at 33.02 83.82 0)
+      (effects (font (size 1.27 1.27)) hide)
+    )
+    (property "Datasheet" "~" (at 33.02 83.82 0)
       (effects (font (size 1.27 1.27)) hide)
     )
@@
         (path "/87282895-5363-4673-9c65-8e036a00088a"
           (reference "H3") (unit 1)
-        )
-      )
-    )
-  )
-  (symbol (lib_id "Connector:TestPoint") (at 121.92 20.32 90) (unit 1)
-    (in_bom no) (on_board yes) (dnp no)
-    (property "Reference" "NE6" (at 123.19 19.05 90)
-      (effects (font (size 1.27 1.27)) (justify left))
-    )
-    (property "Value" "E_E" (at 123.19 16.51 90)
-      (effects (font (size 1.27 1.27)) (justify left))
-    )
-    (property "Footprint" "Surge_Library:NEmount" (at 121.92 15.24 0)
-      (effects (font (size 1.27 1.27)) hide)
-    )
-    (property "Datasheet" "~" (at 121.92 15.24 0)
-      (effects (font (size 1.27 1.27)) hide)
-    )
-    (pin "1")
-    (instances
-      (project "Surge"
-        (path "/87282895-5363-4673-9c65-8e036a00088a"
-          (reference "NE6") (unit 1)
         )
       )
@@
         )
       )
-    )
-  )
-  (symbol (lib_id "Connector:TestPoint") (at 106.68 20.32 270) (unit 1)
-    (in_bom no) (on_board yes) (dnp no)
-    (property "Reference" "NE5" (at 107.95 19.05 90)
-      (effects (font (size 1.27 1.27)) (justify right))
-    )
-    (property "Value" "E_MOV" (at 107.95 16.51 90)
-      (effects (font (size 1.27 1.27)) (justify right))
-    )
-    (property "Footprint" "Surge_Library:NEmount" (at 106.68 25.4 0)
-      (effects (font (size 1.27 1.27)) hide)
-    )
-    (property "Datasheet" "~" (at 106.68 25.4 0)
-      (effects (font (size 1.27 1.27)) hide)
-    )
-    (pin "1")
-    (instances
-      (project "Surge"
-        (path "/87282895-5363-4673-9c65-8e036a00088a"
-          (reference "NE5") (unit 1)
-        )
-      )
