File: Surge.kicad_sch (KiCad schematic)
At the start: 18 parts, among them SW1 C1005B 10A TCB

Commit message: Update Schematics
Parts:
- RV1, RV2, RV3: value 471KD20J -> 471K
- SW1: symbol Switch:SW_DPDT_x2 -> Surge:TCB
- renumbered NE5 to J1, NE4 to J2
Changed lines of the file:
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@@
   (junction (at 100.33 30.48) (diameter 0) (color 0 0 0 0)
+  )
+  (junction (at 56 46.99) (diameter 0) (color 0 0 0 0)
   )
   (junction (at 125.73 45.72) (diameter 0) (color 0 0 0 0)
@@
     (stroke (width 0) (type default))
   )
+  (wire (pts (xy 58.42 60.96) (xy 64.77 60.96))
+    (stroke (width 0) (type default))
+  )
   (wire (pts (xy 35.56 30.48) (xy 41.91 30.48))
     (stroke (width 0) (type default))
@@
     (stroke (width 0) (type dot))
   )
-  (wire (pts (xy 55.88 60.96) (xy 64.77 60.96))
+  (wire (pts (xy 58.42 46.99) (xy 58.42 60.96))
     (stroke (width 0) (type default))
   )
@@
     (stroke (width 0) (type default))
   )
+  (wire (pts (xy 41.91 49.53) (xy 45.72 49.53))
+    (stroke (width 0) (type default))
+  )
   (wire (pts (xy 100.33 81.28) (xy 100.33 83.82))
     (stroke (width 0) (type default))
@@
   )
   (wire (pts (xy 100.33 30.48) (xy 100.33 29.21))
+    (stroke (width 0) (type default))
+  )
+  (wire (pts (xy 56 46.99) (xy 58.42 46.99))
     (stroke (width 0) (type default))
   )
@@
     (stroke (width 0) (type default))
   )
-  (wire (pts (xy 45.72 60.96) (xy 45.72 49.53))
+  (wire (pts (xy 41.91 60.96) (xy 41.91 49.53))
+    (stroke (width 0) (type default))
+  )
+  (wire (pts (xy 55.88 46.99) (xy 56 46.99))
     (stroke (width 0) (type default))
   )
@@
     (stroke (width 0) (type default))
   )
-  (wire (pts (xy 55.88 46.99) (xy 55.88 60.96))
-    (stroke (width 0) (type default))
-  )
-  (wire (pts (xy 35.56 60.96) (xy 45.72 60.96))
+  (wire (pts (xy 35.56 60.96) (xy 41.91 60.96))
     (stroke (width 0) (type default))
   )
@@
       (effects (font (size 1.27 1.27)) (justify left))
     )
-    (property "Value" "471KD20J" (at 102.87 67.5032 0)
+    (property "Value" "471K" (at 102.87 67.5032 0)
       (effects (font (size 1 1)) (justify left))
     )
@@
   (symbol (lib_id "Connector:TestPoint") (at 100.33 71.12 180) (unit 1)
     (in_bom no) (on_board yes) (dnp no)
-    (property "Reference" "NE5" (at 99.06 73.66 0)
+    (property "Reference" "J1" (at 99.06 73.66 0)
       (effects (font (size 1.27 1.27)) (justify left))
     )
@@
       (project "Surge"
         (path "/87282895-5363-4673-9c65-8e036a00088a"
-          (reference "NE5") (unit 1)
+          (reference "J1") (unit 1)
         )
       )
@@
   (symbol (lib_id "Connector:TestPoint") (at 100.33 81.28 0) (unit 1)
     (in_bom no) (on_board yes) (dnp no)
-    (property "Reference" "NE4" (at 99.06 78.74 0)
+    (property "Reference" "J2" (at 99.06 78.74 0)
       (effects (font (size 1.27 1.27)) (justify right))
     )
@@
       (project "Surge"
         (path "/87282895-5363-4673-9c65-8e036a00088a"
-          (reference "NE4") (unit 1)
+          (reference "J2") (unit 1)
         )
       )
@@
       (effects (font (size 1.27 1.27)) (justify left))
     )
-    (property "Value" "471KD20J" (at 102.87 47.1832 0)
+    (property "Value" "471K" (at 102.87 47.1832 0)
       (effects (font (size 1 1)) (justify left))
     )
@@
     )
   )
-  (symbol (lib_id "Switch:SW_DPDT_x2") (at 50.8 46.99 0) (mirror y) (unit 1)
+  (symbol (lib_id "Surge:TCB") (at 50.8 46.99 0) (unit 1)
     (in_bom yes) (on_board yes) (dnp no)
-    (property "Reference" "SW1" (at 52.07 43.18 0)
-      (effects (font (size 1.27 1.27)))
-    )
-    (property "Value" "C1005B 10A TCB" (at 52.07 40.64 0)
-      (effects (font (size 1.27 1.27)))
-    )
-    (property "Footprint" "Surge_Library:Switch" (at 50.8 46.99 0)
-      (effects (font (size 1.27 1.27)) hide)
-    )
-    (property "Datasheet" "~" (at 50.8 46.99 0)
+    (property "Reference" "SW1" (at 52.07 40.64 0)
+      (effects (font (size 1.27 1.27)))
+    )
+    (property "Value" "C1005B 10A TCB" (at 52.07 38.1 0)
+      (effects (font (size 1.27 1.27)))
+    )
+    (property "Footprint" "Surge_Library:Switch" (at 50.8 49.53 0)
+      (effects (font (size 1.27 1.27)) hide)
+    )
+    (property "Datasheet" "~" (at 50.8 49.53 0)
       (effects (font (size 1.27 1.27)) hide)
     )
@@
     (pin "2")
     (pin "3")
-    (pin "4")
-    (pin "5")
-    (pin "6")
     (instances
       (project "Surge"
@@
       (effects (font (size 1.27 1.27)) (justify right))
     )
-    (property "Value" "471KD20J" (at 104.14 26.4766 0)
+    (property "Value" "471K" (at 104.14 26.4766 0)
       (effects (font (size 1 1)) (justify right))
     )

Commit message: Update Readme
Parts:
- N1: renamed from NE1; value Lamp_Neon -> NE2 Bulb
- R1: value 200K Ω -> 100K Ω
- renumbered NE2 to NE1, NE3 to NE2
Changed lines of the file:
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@@
       (effects (font (size 1.27 1.27)))
     )
-    (property "Value" "200K Ω" (at 73.66 41.91 0)
+    (property "Value" "100K Ω" (at 73.66 41.91 0)
       (effects (font (size 1 1)))
     )
@@
   (symbol (lib_id "Device:Lamp_Neon") (at 78.74 49.53 180) (unit 1)
     (in_bom yes) (on_board no) (dnp no)
-    (property "Reference" "NE1" (at 69.85 48.26 0)
-      (effects (font (size 1.27 1.27)))
-    )
-    (property "Value" "Lamp_Neon" (at 69.85 50.4769 0)
+    (property "Reference" "N1" (at 69.85 48.26 0)
+      (effects (font (size 1.27 1.27)))
+    )
+    (property "Value" "NE2 Bulb" (at 69.85 50.4769 0)
       (effects (font (size 1.27 1.27)))
     )
@@
       (project "Surge"
         (path "/87282895-5363-4673-9c65-8e036a00088a"
-          (reference "NE1") (unit 1)
+          (reference "N1") (unit 1)
         )
       )
@@
   (symbol (lib_id "Connector:TestPoint") (at 86.36 54.61 0) (unit 1)
     (in_bom no) (on_board yes) (dnp no) (fields_autoplaced)
-    (property "Reference" "NE3" (at 88.9 50.038 0)
+    (property "Reference" "NE2" (at 88.9 50.038 0)
       (effects (font (size 1.27 1.27)) (justify left))
     )
@@
       (project "Surge"
         (path "/87282895-5363-4673-9c65-8e036a00088a"
-          (reference "NE3") (unit 1)
+          (reference "NE2") (unit 1)
         )
       )
@@
   (symbol (lib_id "Connector:TestPoint") (at 86.36 36.83 180) (unit 1)
     (in_bom no) (on_board yes) (dnp no) (fields_autoplaced)
-    (property "Reference" "NE2" (at 88.9 38.862 0)
+    (property "Reference" "NE1" (at 88.9 38.862 0)
       (effects (font (size 1.27 1.27)) (justify right))
     )
@@
       (project "Surge"
         (path "/87282895-5363-4673-9c65-8e036a00088a"
-          (reference "NE2") (unit 1)
-        )
-      )
+          (reference "NE1") (unit 1)
+        )
+      )
